Commit message: Root the handheld URDF at mid360_link so post_process records odometry as odom -> mid360_link, with base_link its child

File: assets/handheld_recorder.urdf (robot description, URDF)
Before this commit: robot handheld_recorder, 12 links, 11 joints
Links:
- added link mid360_link
Joints:
- added joint mid360_base_joint: type fixed, parent mid360_link, child base_link, origin xyz=0.048656 -0.0001 -0.066976 rpy=-0.436332 0 1.570796

Commit message: Handheld URDF: world -> odom levels base_link (the camera) at the start, and odom -> mid360_link is a floating joint the odometry supplies rather than a static edge

File: assets/handheld_recorder.urdf (robot description, URDF)
Before this commit: robot handheld_recorder, 13 links, 12 joints
Links:
- added link odom
- added link world
Joints:
- added joint odom_mid360_joint: type floating, parent odom, child mid360_link, origin xyz=0 0 0 rpy=0 0 0
- added joint world_odom_joint: type fixed, parent world, child odom, origin xyz=0.0001 0.015792 0.081263 rpy=0 0.436332 -1.570796
